File: mask-0.0.0/mask-0.0.0.kicad_sch (KiCad schematic)
At the start: 0 parts

Commit message: copy cherry mx libs for Kailh Socket mod
Parts:
- added SW1: SW_Push, Button_Switch_Keyboard:SW_Cherry_MX_1.00u_PCB, symbol Switch:SW_Push
Changed lines of the file:
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@@
-(kicad_sch (version 20210126) (generator eeschema)
+(kicad_sch (version 20210621) (generator eeschema)
   (paper "A4")
-  (symbol_instances)
+  (symbol (lib_id "Switch:SW_Push") (at 86.36 40.64 0) (unit 1)
+    (in_bom yes) (on_board yes) (fields_autoplaced)
+    (property "Reference" "SW1" (id 0) (at 86.36 33.7524 0))
+    (property "Value" "SW_Push" (id 1) (at 86.36 36.5275 0))
+    (property "Footprint" "Button_Switch_Keyboard:SW_Cherry_MX_1.00u_PCB" (id 2) (at 86.36 35.56 0)
+      (effects (font (size 1.27 1.27)) hide)
+    )
+    (property "Datasheet" "~" (id 3) (at 86.36 35.56 0)
+      (effects (font (size 1.27 1.27)) hide)
+    )
+    (pin "1")
+    (pin "2")
+  )
+  (sheet_instances
+    (path "/" (page "1"))
+  )
+  (symbol_instances
+    (path "/2f33e429-a91b-408b-b315-3ebb0c8951f5"
+      (reference "SW1") (unit 1) (value "SW_Push") (footprint "Button_Switch_Keyboard:SW_Cherry_MX_1.00u_PCB")
+    )
+  )
 )
