File: mask-0.0.0/mask-0.0.0.kicad_pcb (KiCad board)
At the start: 2 copper layers, 0 parts

Commit message: draw basic key-matrix
Parts:
- added D1: 1N4148W, Diode_SMD:D_SOD-123, F.Cu at (117.2, 180.4)
- added D10: 1N4148W, Diode_SMD:D_SOD-123, F.Cu at (111.5, 180.4)
- added D11: 1N4148W, Diode_SMD:D_SOD-123, F.Cu at (140.2, 183.8)
- added D12: 1N4148W, Diode_SMD:D_SOD-123, F.Cu at (11.6, 72.1)
- added D13: 1N4148W, Diode_SMD:D_SOD-123, F.Cu at (71.2, 180.4)
- added D14: 1N4148W, Diode_SMD:D_SOD-123, F.Cu at (100.0, 183.8)
- added D15: 1N4148W, Diode_SMD:D_SOD-123, F.Cu at (77.0, 183.8)
- added D16: 1N4148W, Diode_SMD:D_SOD-123, F.Cu at (105.8, 180.4)
- added D17: 1N4148W, Diode_SMD:D_SOD-123, F.Cu at (88.5, 183.8)
- added D18: 1N4148W, Diode_SMD:D_SOD-123, F.Cu at (-8.56, 92.3)
- added D19: 1N4148W, Diode_SMD:D_SOD-123, F.Cu at (100.0, 180.4)
- added D2: 1N4148W, Diode_SMD:D_SOD-123, F.Cu at (146.0, 183.8)
- added D20: 1N4148W, Diode_SMD:D_SOD-123, F.Cu at (140.2, 180.4)
- added D21: 1N4148W, Diode_SMD:D_SOD-123, F.Cu at (151.8, 180.4)
- added D22: 1N4148W, Diode_SMD:D_SOD-123, F.Cu at (111.5, 183.8)
- added D23: 1N4148W, Diode_SMD:D_SOD-123, F.Cu at (94.2, 180.4)
- added D24: 1N4148W, Diode_SMD:D_SOD-123, F.Cu at (104.4, 92.9)
- added D25: 1N4148W, Diode_SMD:D_SOD-123, F.Cu at (128.8, 183.8)
- added D26: 1N4148W, Diode_SMD:D_SOD-123, F.Cu at (77.0, 180.4)
- added D27: 1N4148W, Diode_SMD:D_SOD-123, F.Cu at (-28.8, 115.8)
- added D28: 1N4148W, Diode_SMD:D_SOD-123, F.Cu at (123.0, 180.4)
- added D29: 1N4148W, Diode_SMD:D_SOD-123, F.Cu at (94.2, 183.8)
- added D3: 1N4148W, Diode_SMD:D_SOD-123, F.Cu at (-28.8, 112.5)
- added D30: 1N4148W, Diode_SMD:D_SOD-123, F.Cu at (88.5, 180.4)
- added D31: 1N4148W, Diode_SMD:D_SOD-123, F.Cu at (134.5, 180.4)
- added D32: 1N4148W, Diode_SMD:D_SOD-123, F.Cu at (71.2, 183.8)
- added D33: 1N4148W, Diode_SMD:D_SOD-123, F.Cu at (105.8, 183.8)
- added D34: 1N4148W, Diode_SMD:D_SOD-123, F.Cu at (128.8, 180.4)
- added D35: 1N4148W, Diode_SMD:D_SOD-123, F.Cu at (82.8, 180.4)
- added D4: 1N4148W, Diode_SMD:D_SOD-123, F.Cu at (134.5, 183.8)
- added D5: 1N4148W, Diode_SMD:D_SOD-123, F.Cu at (146.0, 180.4)
- added D6: 1N4148W, Diode_SMD:D_SOD-123, F.Cu at (238.2, 51.6)
- added D7: 1N4148W, Diode_SMD:D_SOD-123, F.Cu at (123.0, 183.8)
- added D8: 1N4148W, Diode_SMD:D_SOD-123, F.Cu at (117.2, 183.8)
- added D9: 1N4148W, Diode_SMD:D_SOD-123, F.Cu at (82.8, 183.8)
- added SW1: SW_Push, Button_Switch_Keyboard_Swappable:SW_Cherry_MX_1.00u_Kailh_Socket_TopBottom, F.Cu at (75.0, 25.0)
- added SW10: SW_Push, Button_Switch_Keyboard_Swappable:SW_Cherry_MX_1.00u_Kailh_Socket_TopBottom, F.Cu at (115.0, 45.0)
- added SW11: SW_Push, Button_Switch_Keyboard_Swappable:SW_Cherry_MX_1.00u_Kailh_Socket_TopBottom, F.Cu at (135.0, 45.0)
- added SW12: SW_Push, Button_Switch_Keyboard_Swappable:SW_Cherry_MX_1.00u_Kailh_Socket_TopBottom, F.Cu at (155.0, 45.0)
- added SW13: SW_Push, Button_Switch_Keyboard_Swappable:SW_Cherry_MX_1.00u_Kailh_Socket_TopBottom, F.Cu at (175.0, 45.0)
- added SW14: SW_Push, Button_Switch_Keyboard_Swappable:SW_Cherry_MX_1.00u_Kailh_Socket_TopBottom, F.Cu at (195.0, 45.0)
- added SW15: SW_Push, Button_Switch_Keyboard_Swappable:SW_Cherry_MX_1.00u_Kailh_Socket_TopBottom, F.Cu at (75.0, 65.0)
- added SW16: SW_Push, Button_Switch_Keyboard_Swappable:SW_Cherry_MX_1.00u_Kailh_Socket_TopBottom, F.Cu at (95.0, 65.0)
- added SW17: SW_Push, Button_Switch_Keyboard_Swappable:SW_Cherry_MX_1.00u_Kailh_Socket_TopBottom, F.Cu at (115.0, 65.0)
- added SW18: SW_Push, Button_Switch_Keyboard_Swappable:SW_Cherry_MX_1.00u_Kailh_Socket_TopBottom, F.Cu at (135.0, 65.0)
- added SW19: SW_Push, Button_Switch_Keyboard_Swappable:SW_Cherry_MX_1.00u_Kailh_Socket_TopBottom, F.Cu at (155.0, 65.0)
- added SW2: SW_Push, Button_Switch_Keyboard_Swappable:SW_Cherry_MX_1.00u_Kailh_Socket_TopBottom, F.Cu at (95.0, 25.0)
- added SW20: SW_Push, Button_Switch_Keyboard_Swappable:SW_Cherry_MX_1.00u_Kailh_Socket_TopBottom, F.Cu at (175.0, 65.0)
- added SW21: SW_Push, Button_Switch_Keyboard_Swappable:SW_Cherry_MX_1.00u_Kailh_Socket_TopBottom, F.Cu at (195.0, 65.0)
- added SW22: SW_Push, Button_Switch_Keyboard_Swappable:SW_Cherry_MX_1.00u_Kailh_Socket_TopBottom, F.Cu at (75.0, 85.0)
- added SW23: SW_Push, Button_Switch_Keyboard_Swappable:SW_Cherry_MX_1.00u_Kailh_Socket_TopBottom, F.Cu at (95.0, 85.0)
- added SW24: SW_Push, Button_Switch_Keyboard_Swappable:SW_Cherry_MX_1.00u_Kailh_Socket_TopBottom, F.Cu at (115.0, 85.0)
- added SW25: SW_Push, Button_Switch_Keyboard_Swappable:SW_Cherry_MX_1.00u_Kailh_Socket_TopBottom, F.Cu at (135.0, 85.0)
- added SW26: SW_Push, Button_Switch_Keyboard_Swappable:SW_Cherry_MX_1.00u_Kailh_Socket_TopBottom, F.Cu at (155.0, 85.0)
- added SW27: SW_Push, Button_Switch_Keyboard_Swappable:SW_Cherry_MX_1.00u_Kailh_Socket_TopBottom, F.Cu at (175.0, 85.0)
- added SW28: SW_Push, Button_Switch_Keyboard_Swappable:SW_Cherry_MX_1.00u_Kailh_Socket_TopBottom, F.Cu at (195.0, 85.0)
- added SW29: SW_Push, Button_Switch_Keyboard_Swappable:SW_Cherry_MX_1.00u_Kailh_Socket_TopBottom, F.Cu at (75.0, 105.0)
- added SW3: SW_Push, Button_Switch_Keyboard_Swappable:SW_Cherry_MX_1.00u_Kailh_Socket_TopBottom, F.Cu at (115.0, 25.0)
- added SW30: SW_Push, Button_Switch_Keyboard_Swappable:SW_Cherry_MX_1.00u_Kailh_Socket_TopBottom, F.Cu at (95.0, 105.0)
- added SW31: SW_Push, Button_Switch_Keyboard_Swappable:SW_Cherry_MX_1.00u_Kailh_Socket_TopBottom, F.Cu at (115.0, 105.0)
- added SW32: SW_Push, Button_Switch_Keyboard_Swappable:SW_Cherry_MX_1.00u_Kailh_Socket_TopBottom, F.Cu at (135.0, 105.0)
- added SW33: SW_Push, Button_Switch_Keyboard_Swappable:SW_Cherry_MX_1.00u_Kailh_Socket_TopBottom, F.Cu at (155.0, 105.0)
- added SW34: SW_Push, Button_Switch_Keyboard_Swappable:SW_Cherry_MX_1.00u_Kailh_Socket_TopBottom, F.Cu at (175.0, 105.0)
- added SW35: SW_Push, Button_Switch_Keyboard_Swappable:SW_Cherry_MX_1.00u_Kailh_Socket_TopBottom, F.Cu at (195.0, 105.0)
- added SW4: SW_Push, Button_Switch_Keyboard_Swappable:SW_Cherry_MX_1.00u_Kailh_Socket_TopBottom, F.Cu at (135.0, 25.0)
- added SW5: SW_Push, Button_Switch_Keyboard_Swappable:SW_Cherry_MX_1.00u_Kailh_Socket_TopBottom, F.Cu at (155.0, 25.0)
- added SW6: SW_Push, Button_Switch_Keyboard_Swappable:SW_Cherry_MX_1.00u_Kailh_Socket_TopBottom, F.Cu at (175.0, 25.0)
- added SW7: SW_Push, Button_Switch_Keyboard_Swappable:SW_Cherry_MX_1.00u_Kailh_Socket_TopBottom, F.Cu at (195.0, 25.0)
- added SW8: SW_Push, Button_Switch_Keyboard_Swappable:SW_Cherry_MX_1.00u_Kailh_Socket_TopBottom, F.Cu at (75.0, 45.0)
- added SW9: SW_Push, Button_Switch_Keyboard_Swappable:SW_Cherry_MX_1.00u_Kailh_Socket_TopBottom, F.Cu at (95.0, 45.0)

Commit message: change diodes package, start test positioning in correct distance
Parts:
- added REF**: SW_Cherry_MX_2.00u_PCB, Button_Switch_Keyboard_Swappable:SW_Cherry_MX_2.00u_Kailh_Socket_TopBottom, F.Cu at (177.3, 122.1)
- added REF**: SW_Cherry_MX_1.75u_PCB, Button_Switch_Keyboard_Swappable:SW_Cherry_MX_1.75u_Kailh_Socket_TopBottom, F.Cu at (112.0, 165.9)
- added REF**: SW_Cherry_MX_1.75u_PCB, Button_Switch_Keyboard_Swappable:SW_Cherry_MX_1.75u_Kailh_Socket_TopBottom, F.Cu at (178.7, 165.9)
- added REF**: SW_Cherry_MX_1.75u_PCB, Button_Switch_Keyboard_Swappable:SW_Cherry_MX_1.75u_Kailh_Socket_TopBottom, F.Cu at (145.4, 165.9)
- added REF**: SW_Cherry_MX_1.75u_PCB, Button_Switch_Keyboard_Swappable:SW_Cherry_MX_1.75u_Kailh_Socket_TopBottom, F.Cu at (78.7, 165.9)
- D1, D10, D11, D12, D13, D14, D15, D16, D17, D18, D19, D2, D20, D21, D22, D23, D24, D25, D26, D27, D28, D29, D3, D30, D31, D32, D33, D34, D35, D4, D5, D6, D7, D8, D9: footprint Diode_SMD:D_SOD-123 -> Diode_SMD_TopBottom:D_SOD-123_TopBottom
- moved D27 194.2 mm to (161.0, 157.0), turned to -90 degrees
- moved D3 152.5 mm to (116.9, 67.4), turned to -90 degrees
- moved D18 145.1 mm to (135.8, 106.1), turned to -90 degrees
- moved D12 143.4 mm to (154.3, 86.5), turned to -90 degrees
- moved D13 138.5 mm to (173.7, 87.2), turned to -90 degrees
- moved D7 135.8 mm to (192.2, 67.0), turned to -90 degrees
- moved D14 134.0 mm to (192.2, 86.6), turned to -90 degrees
- moved D2 126.1 mm to (97.8, 67.3), turned to -90 degrees
- moved D1 119.9 mm to (79.3, 66.7), turned to -90 degrees
- moved D4 116.3 mm to (135.3, 67.5), turned to -90 degrees
- moved D5 113.2 mm to (154.4, 67.5), turned to -90 degrees
- moved D8 105.2 mm to (78.4, 86.1), turned to -90 degrees
- moved D9 98.9 mm to (97.3, 86.0), turned to -90 degrees
- moved D11 97.5 mm to (135.5, 86.4), turned to -90 degrees
- moved D26 95.4 mm to (154.6, 125.0), turned to -90 degrees
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Connections:
- D13 pad 1: /ROW0 -> /ROW1
- D13 pad 2: Net-(SW7-Pad2) -> Net-(SW13-Pad2)
- D7 pad 1: /ROW1 -> /ROW0
- D8 pad 2: Net-(SW9-Pad2) -> Net-(SW8-Pad2)
- D9 pad 2: Net-(SW10-Pad2) -> Net-(D9-Pad2)
- SW10 pad 2: Net-(SW10-Pad2) -> Net-(D10-Pad2)
- SW11 pad 2: Net-(D10-Pad2) -> Net-(D11-Pad2)
- SW12 pad 2: Net-(D11-Pad2) -> Net-(D12-Pad2)
- SW13 pad 2: Net-(D12-Pad2) -> Net-(SW13-Pad2)
- SW7 pad 2: Net-(SW7-Pad2) -> Net-(D7-Pad2)
- SW8 pad 2: Net-(D7-Pad2) -> Net-(SW8-Pad2)
- SW9 pad 2: Net-(SW9-Pad2) -> Net-(D9-Pad2)

Commit message: test-place buttons (only ortholinear, not shifted)
Parts:
- removed REF**: SW_Cherry_MX_2.00u_PCB, Button_Switch_Keyboard_Swappable:SW_Cherry_MX_2.00u_Kailh_Socket_TopBottom
- removed REF** (x4): SW_Cherry_MX_1.75u_PCB, Button_Switch_Keyboard_Swappable:SW_Cherry_MX_1.75u_Kailh_Socket_TopBottom
- added SW13_1: SW_Push, Button_Switch_Keyboard_Swappable:SW_Cherry_MX_2.00u_Kailh_Socket_NoStabilizer_TopBottom, F.Cu at (177.3, 84.0)
- added SW20_1: SW_Push, Button_Switch_Keyboard_Swappable:SW_Cherry_MX_2.00u_Kailh_Socket_NoStabilizer_TopBottom, F.Cu at (177.3, 103.0)
- added SW27_1: SW_Push, Button_Switch_Keyboard_Swappable:SW_Cherry_MX_2.00u_Kailh_Socket_NoStabilizer_TopBottom, F.Cu at (177.3, 122.1)
- SW31, SW32, SW33, SW34, SW35: footprint Button_Switch_Keyboard_Swappable:SW_Cherry_MX_1.00u_Kailh_Socket_TopBottom -> Button_Switch_Keyboard_Swappable:SW_Cherry_MX_1.50u_Kailh_Socket_TopBottom
- moved D27 43.3 mm to (189.2, 124.2)
- moved D35 41.0 mm to (190.1, 144.6)
- moved SW35 38.6 mm to (177.0, 151.3)
- moved D34 34.7 mm to (161.9, 144.5)
- moved SW34 32.1 mm to (148.4, 151.3)
- moved D28 32.0 mm to (191.7, 124.1)
- moved D33 28.6 mm to (133.4, 144.5)
- moved SW33 26.5 mm to (119.8, 151.3)
- moved D32 23.8 mm to (105.2, 144.5)
- moved SW32 21.0 mm to (91.3, 151.3)
- moved D31 18.8 mm to (77.6, 144.6)
- moved D20 16.5 mm to (190.4, 104.8)
- moved D13 15.8 mm to (189.5, 86.5)
- moved SW31 15.5 mm to (62.7, 151.3)
Other:
- board outline added: 143.4 x 111.5 mm

Commit message: first test layout
Parts:
- SW31: footprint Button_Switch_Keyboard_Swappable:SW_Cherry_MX_1.50u_Kailh_Socket_TopBottom -> Button_Switch_Keyboard_Swappable:SW_Cherry_MX_1.25u_Kailh_Socket_TopBottom
- SW32, SW33, SW34, SW35: footprint Button_Switch_Keyboard_Swappable:SW_Cherry_MX_1.50u_Kailh_Socket_TopBottom -> Button_Switch_Keyboard_Swappable:SW_Cherry_MX_1.00u_Kailh_Socket_TopBottom
- moved D35 56.7 mm to (133.5, 142.0)
- moved SW35 53.0 mm to (124.0, 151.3)
- moved D34 47.9 mm to (114.0, 142.5)
- moved SW34 43.7 mm to (104.7, 151.3)
- moved D33 39.9 mm to (93.5, 144.5)
- moved SW33 37.4 mm to (82.5, 154.0), turned to -176 degrees
- moved D32 33.8 mm to (71.5, 146.5)
- moved D31 30.1 mm to (47.5, 144.0), turned to 0 degrees
- moved SW32 29.5 mm to (62.4, 157.3), turned to -168 degrees
- moved SW31 25.7 mm to (37.2, 154.6), turned to 110 degrees
- moved D7 5.54 mm to (192.5, 72.5)
- moved D6 5.03 mm to (173.5, 72.5)
- moved D5 4.95 mm to (154.5, 72.5)
- moved D19 4.90 mm to (154.5, 110.0)
- moved SW13_1 4.56 mm to (177.3, 88.5)
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Other:
- board size 143.4 x 111.5 mm -> 165 x 113 mm
