File: mask-0.0.0/keymatrix.kicad_sch (KiCad schematic)
At the start: 73 parts, among them SW1 SW_Push, SW10 SW_Push, SW11 SW_Push, SW12 SW_Push, SW13 SW_Push, SW13_1 SW_Push, SW14 SW_Push, SW15 SW_Push, SW16 SW_Push, SW17 SW_Push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

Commit message: udpate routing
Parts:
- renumbered D22 to D10, D29 to D11, D2 to D12, D9 to D13, D16 to D14, D23 to D15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

Commit message: mask-0.0.0: begin of matrix routing
Parts:
- renumbered SW8 to SW10, SW9 to SW11, SW10 to SW12, SW11 to SW13, SW12 to SW14, SW13 to SW15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
