File: mask-2.0.0/mask-2.0.0.kicad_pcb (KiCad board)
At the start: 2 copper layers, 307.3 x 148.3 mm, 161 parts, among them J1 USB_C_Receptacle_USB2.0, J2 Conn_01x04, J3 Conn_01x04, SW1 Cherry_MX_ULP_SK6812_1515, SW10 Cherry_MX_ULP_SK6812_1515, SW11 Cherry_MX_ULP_SK6812_1515, SW12 Cherry_MX_ULP_SK6812_1515, SW13 Cherry_MX_ULP_SK6812_1515, SW14 Cherry_MX_ULP_SK6812_1515, SW15 Cherry_MX_ULP_SK6812_1515, SW16 Cherry_MX_ULP_SK6812_1515, SW17 Cherry_MX_ULP_SK6812_1515, SW18 Cherry_MX_ULP_SK6812_1515, SW19 Cherry_MX_ULP_SK6812_1515, SW2 Cherry_MX_ULP_SK6812_1515, SW20 Cherry_MX_ULP_SK6812_1515, SW21 Cherry_MX_ULP_SK6812_1515, SW22 Cherry_MX_ULP_SK6812_1515, SW23 Cherry_MX_ULP_SK6812_1515, SW24 Cherry_MX_ULP_SK6812_1515, SW25 Cherry_MX_ULP_SK6812_1515, SW26 Cherry_MX_ULP_SK6812_1515, SW27 Cherry_MX_ULP_SK6812_1515, SW28 Cherry_MX_ULP_SK6812_1515, SW29 Cherry_MX_ULP_SK6812_1515, SW3 Cherry_MX_ULP_SK6812_1515, SW30 Cherry_MX_ULP_SK6812_1515, SW31 Cherry_MX_ULP_SK6812_1515, SW32 Cherry_MX_ULP_SK6812_1515, SW33 Cherry_MX_ULP_SK6812_1515, SW34 Cherry_MX_ULP_SK6812_1515, SW35 Cherry_MX_ULP_SK6812_1515, SW36 Cherry_MX_ULP_SK6812_1515, SW37 Cherry_MX_ULP_SK6812_1515, SW38 Cherry_MX_ULP_SK6812_1515, SW39 Cherry_MX_ULP_SK6812_1515, SW4 Cherry_MX_ULP_SK6812_1515, SW40 Cherry_MX_ULP_SK6812_1515, SW41 Cherry_MX_ULP_SK6812_1515, SW42 Cherry_MX_ULP_SK6812_1515, SW43 Cherry_MX_ULP_SK6812_1515, SW44 Cherry_MX_ULP_SK6812_1515, SW45 Cherry_MX_ULP_SK6812_1515, SW46 Cherry_MX_ULP_SK6812_1515, SW47 Cherry_MX_ULP_SK6812_1515, SW48 Cherry_MX_ULP_SK6812_1515, SW49 Cherry_MX_ULP_SK6812_1515, SW5 Cherry_MX_ULP_SK6812_1515, SW50 Cherry_MX_ULP_SK6812_1515, SW51 Cherry_MX_ULP_SK6812_1515, SW52 Cherry_MX_ULP_SK6812_1515, SW53 Cherry_MX_ULP_SK6812_1515, SW54 Cherry_MX_ULP_SK6812_1515, SW55 Cherry_MX_ULP_SK6812_1515, SW56 Cherry_MX_ULP_SK6812_1515, SW57 Cherry_MX_ULP_SK6812_1515, SW58 Cherry_MX_ULP_SK6812_1515, SW59 Cherry_MX_ULP_SK6812_1515, SW6 Cherry_MX_ULP_SK6812_1515, SW60 Cherry_MX_ULP_SK6812_1515, SW61 SW_Push, SW62 SW_Push, SW7 Cherry_MX_ULP_SK6812_1515, SW8 Cherry_MX_ULP_SK6812_1515, SW9 Cherry_MX_ULP_SK6812_1515, U1 RP2040, U2 AP2112K-3.3, U3 W25Q128JVPIQ, Y1 445C25D12M00000

Commit message: mask-2.0.0: update to smd kb2040 variant
Parts:
- removed C10, C20, C21: 1uF, Capacitor_SMD:C_0603_1608Metric
- removed C11, C12, C13, C14, C15, C16, C17, C18, C19, C6, C7: 100nF, Capacitor_SMD:C_0603_1608Metric
- removed C3: 10nF, Capacitor_SMD:C_0603_1608Metric
- removed C4: 10pF, Capacitor_SMD:C_0603_1608Metric
- removed C5: 10uF, Capacitor_SMD:C_0805_2012Metric
- removed C8, C9: 22pF, Capacitor_SMD:C_0603_1608Metric
- removed the D10 at (237.0, 39.5)
- removed the D11 at (256.0, 39.5)
- removed the D12 at (275.5, 39.5)
- removed the D19 at (335.0, 74.3)
- removed the D20 at (388.5, 65.2)
- removed the D21 at (335.0, 77.7)
- removed the D22 at (353.0, 73.0)
- removed the D23 at (338.5, 56.0)
- removed the D24 at (403.5, 73.5)
- removed D31, D32, D33, D34, D35, D36, D43, D44, D45, D46, D47, D48, D55, D56, D57, D58, D59, D60: 1N4148W, Diode_SMD:D_SOD-123
- removed D61: PRTR5V0U2X, Package_TO_SOT_SMD:SOT-143
- removed D62: LED, LED_SMD:LED_0603_1608Metric
- removed the D7 at (180.5, 39.5)
- removed the D8 at (199.5, 39.5)
- removed the D9 at (218.0, 39.5)
- removed FB1: 120R@550mA, Resistor_SMD:R_0603_1608Metric
- removed the J3 at (376.7, 35.7)
- removed the SW10 at (237.0, 30.0)
- removed the SW11 at (256.0, 30.0)
- removed the SW12 at (275.0, 30.0)
- removed the SW19 at (180.0, 49.0)
- removed the SW20 at (199.0, 49.0)
- removed the SW21 at (218.0, 49.0)
- removed the SW22 at (237.0, 49.0)
- removed the SW23 at (256.0, 49.0)
- removed the SW24 at (275.0, 49.0)
- removed the SW31 at (180.0, 68.0)
- removed the SW32 at (199.0, 68.0)
- removed SW33, SW34, SW35, SW36, SW43, SW44, SW45, SW46, SW47, SW48, SW55, SW56, SW57, SW58, SW59, SW60: Cherry_MX_ULP_SK6812_1515, mask:Cherry_MX_ULP_SK6812_1515
- removed SW61: SW_Push, Button_Switch_SMD:SW_SPST_B3U-1000P
- removed the SW7 at (180.0, 30.0)
- removed the SW8 at (199.0, 30.0)
- removed the SW9 at (218.0, 30.0)
- removed U2: AP2112K-3.3, Package_TO_SOT_SMD:SOT-23-5
- removed U3: W25Q128JVPIQ, Package_SON:WSON-8-1EP_6x5mm_P1.27mm_EP3.4x4.3mm
- removed Y1: 445C25D12M00000, Crystal:Crystal_SMD_5032-2Pin_5.0x3.2mm
- added J2: USB_C_Receptacle_USB2.0, Connector_USB:USB_C_Receptacle_JAE_DX07S016JA1R1500, F.Cu at (182.0, 72.0)
- added JP1: SolderJumper_3_Bridged12, Jumper:SolderJumper-3_P1.3mm_Bridged12_RoundedPad1.0x1.5mm_NumberLabels, F.Cu at (258.5, 104.0)
- added JP2: SolderJumper_3_Bridged12, Jumper:SolderJumper-3_P1.3mm_Bridged12_RoundedPad1.0x1.5mm_NumberLabels, F.Cu at (258.4, 108.7)
- added JP3: SolderJumper_2_Open, Jumper:SolderJumper-2_P1.3mm_Open_RoundedPad1.0x1.5mm, F.Cu at (291.0, 73.1)
- added JP4: SolderJumper_2_Open, Jumper:SolderJumper-2_P1.3mm_Open_RoundedPad1.0x1.5mm, F.Cu at (291.6, 77.5)
- added SW26: SW_Push, Button_Switch_SMD:SW_SPST_B3U-1000P, F.Cu at (210.5, 88.0)
- C1: value 10uF -> 100nF; footprint Capacitor_SMD:C_0805_2012Metric -> Capacitor_SMD:C_0603_1608Metric
- C2: value 10nF -> 100nF
- D1, D2, D3, D4, D5, D6: footprint Diode_SMD:D_SOD-123 -> mask:D_SOD-123_TopBottom
- D10: renamed from D16; footprint Diode_SMD:D_SOD-123 -> mask:D_SOD-123_TopBottom
- D11: renamed from D17; footprint Diode_SMD:D_SOD-123 -> mask:D_SOD-123_TopBottom
- D12: renamed from D18; footprint Diode_SMD:D_SOD-123 -> mask:D_SOD-123_TopBottom
- D13: renamed from D25; footprint Diode_SMD:D_SOD-123 -> mask:D_SOD-123_TopBottom
- D14: renamed from D26; footprint Diode_SMD:D_SOD-123 -> mask:D_SOD-123_TopBottom
- D15: renamed from D27; footprint Diode_SMD:D_SOD-123 -> mask:D_SOD-123_TopBottom
- D16: renamed from D28; footprint Diode_SMD:D_SOD-123 -> mask:D_SOD-123_TopBottom
- D17: renamed from D29; footprint Diode_SMD:D_SOD-123 -> mask:D_SOD-123_TopBottom
- D18: renamed from D30; footprint Diode_SMD:D_SOD-123 -> mask:D_SOD-123_TopBottom
- D19: renamed from D37; footprint Diode_SMD:D_SOD-123 -> mask:D_SOD-123_TopBottom
- D20: renamed from D38; footprint Diode_SMD:D_SOD-123 -> mask:D_SOD-123_TopBottom
- D21: renamed from D39; footprint Diode_SMD:D_SOD-123 -> mask:D_SOD-123_TopBottom
- D22: renamed from D40; footprint Diode_SMD:D_SOD-123 -> mask:D_SOD-123_TopBottom
- D23: renamed from D41; footprint Diode_SMD:D_SOD-123 -> mask:D_SOD-123_TopBottom
- D24: renamed from D42; footprint Diode_SMD:D_SOD-123 -> mask:D_SOD-123_TopBottom
- D25: renamed from D49; footprint Diode_SMD:D_SOD-123 -> mask:D_SOD-123_TopBottom
- D26: renamed from D50; footprint Diode_SMD:D_SOD-123 -> mask:D_SOD-123_TopBottom
- D27: renamed from D51; footprint Diode_SMD:D_SOD-123 -> mask:D_SOD-123_TopBottom
- D28: renamed from D52; footprint Diode_SMD:D_SOD-123 -> mask:D_SOD-123_TopBottom
- D29: renamed from D53; footprint Diode_SMD:D_SOD-123 -> mask:D_SOD-123_TopBottom
- D30: renamed from D54; footprint Diode_SMD:D_SOD-123 -> mask:D_SOD-123_TopBottom
- D7: renamed from D13; footprint Diode_SMD:D_SOD-123 -> mask:D_SOD-123_TopBottom
- D8: renamed from D14; footprint Diode_SMD:D_SOD-123 -> mask:D_SOD-123_TopBottom
- D9: renamed from D15; footprint Diode_SMD:D_SOD-123 -> mask:D_SOD-123_TopBottom
- J1: moved to B.Cu
- R2, R3: value 27 -> 1k
- R4: value 5.1k -> 1k
- R5: value 5.1k -> 2.2k
- R6, R8: value 10k -> 2.2k
- R7: value 1k -> 2.2k
- SW1, SW2, SW3, SW4, SW5, SW6: footprint mask:Cherry_MX_ULP_SK6812_1515 -> mask:Cherry_MX_ULP_SK6812_1515_TopBottom
- SW10: renamed from SW16; footprint mask:Cherry_MX_ULP_SK6812_1515 -> mask:Cherry_MX_ULP_SK6812_1515_TopBottom
- SW11: renamed from SW17; footprint mask:Cherry_MX_ULP_SK6812_1515 -> mask:Cherry_MX_ULP_SK6812_1515_TopBottom
- SW12: renamed from SW18; footprint mask:Cherry_MX_ULP_SK6812_1515 -> mask:Cherry_MX_ULP_SK6812_1515_TopBottom
- SW13: renamed from SW25; footprint mask:Cherry_MX_ULP_SK6812_1515 -> mask:Cherry_MX_ULP_SK6812_1515_TopBottom
- SW14: renamed from SW26; footprint mask:Cherry_MX_ULP_SK6812_1515 -> mask:Cherry_MX_ULP_SK6812_1515_TopBottom
- SW15: renamed from SW27; footprint mask:Cherry_MX_ULP_SK6812_1515 -> mask:Cherry_MX_ULP_SK6812_1515_TopBottom
- SW16: renamed from SW28; footprint mask:Cherry_MX_ULP_SK6812_1515 -> mask:Cherry_MX_ULP_SK6812_1515_TopBottom
- SW17: renamed from SW29; footprint mask:Cherry_MX_ULP_SK6812_1515 -> mask:Cherry_MX_ULP_SK6812_1515_TopBottom
- SW18: renamed from SW30; footprint mask:Cherry_MX_ULP_SK6812_1515 -> mask:Cherry_MX_ULP_SK6812_1515_TopBottom
- SW19: renamed from SW37; footprint mask:Cherry_MX_ULP_SK6812_1515 -> mask:Cherry_MX_ULP_SK6812_1515_TopBottom
- SW20: renamed from SW38; footprint mask:Cherry_MX_ULP_SK6812_1515 -> mask:Cherry_MX_ULP_SK6812_1515_TopBottom
- SW21: renamed from SW39; footprint mask:Cherry_MX_ULP_SK6812_1515 -> mask:Cherry_MX_ULP_SK6812_1515_TopBottom
- SW22: renamed from SW40; footprint mask:Cherry_MX_ULP_SK6812_1515 -> mask:Cherry_MX_ULP_SK6812_1515_TopBottom
- SW23: renamed from SW41; footprint mask:Cherry_MX_ULP_SK6812_1515 -> mask:Cherry_MX_ULP_SK6812_1515_TopBottom
- SW24: renamed from SW42; footprint mask:Cherry_MX_ULP_SK6812_1515 -> mask:Cherry_MX_ULP_SK6812_1515_TopBottom
- SW27: renamed from SW49; footprint mask:Cherry_MX_ULP_SK6812_1515 -> mask:Cherry_MX_ULP_SK6812_1515_TopBottom
- SW28: renamed from SW50; footprint mask:Cherry_MX_ULP_SK6812_1515 -> mask:Cherry_MX_ULP_SK6812_1515_TopBottom
- SW29: renamed from SW51; footprint mask:Cherry_MX_ULP_SK6812_1515 -> mask:Cherry_MX_ULP_SK6812_1515_TopBottom
- SW30: renamed from SW52; footprint mask:Cherry_MX_ULP_SK6812_1515 -> mask:Cherry_MX_ULP_SK6812_1515_TopBottom
- SW31: renamed from SW53; footprint mask:Cherry_MX_ULP_SK6812_1515 -> mask:Cherry_MX_ULP_SK6812_1515_TopBottom
- SW32: renamed from SW54; footprint mask:Cherry_MX_ULP_SK6812_1515 -> mask:Cherry_MX_ULP_SK6812_1515_TopBottom
- SW7: renamed from SW13; footprint mask:Cherry_MX_ULP_SK6812_1515 -> mask:Cherry_MX_ULP_SK6812_1515_TopBottom
- SW8: renamed from SW14; footprint mask:Cherry_MX_ULP_SK6812_1515 -> mask:Cherry_MX_ULP_SK6812_1515_TopBottom
- SW9: renamed from SW15; footprint mask:Cherry_MX_ULP_SK6812_1515 -> mask:Cherry_MX_ULP_SK6812_1515_TopBottom
- U1: value RP2040 -> ProMicro; footprint Package_DFN_QFN:QFN-56-1EP_7x7mm_P0.4mm_EP3.2x3.2mm -> mask:KB2040_SMD
- moved R5 228.5 mm to (162.5, 69.0), turned to 0 degrees
- moved R8 228.3 mm to (162.0, 72.5), turned to 0 degrees
- moved R7 226.0 mm to (166.0, 71.5), turned to 0 degrees
- moved R1 222.2 mm to (179.5, 81.0), turned to 180 degrees
- moved R6 222.1 mm to (166.5, 69.0), turned to 0 degrees
- moved R2 220.5 mm to (183.0, 83.5), turned to 0 degrees
- moved C1 210.3 mm to (179.5, 83.5), turned to 0 degrees
- moved C2 209.9 mm to (187.0, 83.5), turned to 0 degrees
- moved J3 208.6 mm to (165.2, 63.5), turned to 90 degrees
- moved R3 190.2 mm to (204.3, 85.3), turned to 0 degrees
- moved U1 189.4 mm to (169.2, 40.0)
- moved R4 189.1 mm to (210.5, 85.0), turned to 0 degrees
- moved D15 181.0 mm to (198.3, 120.1)
- moved D26 181.0 mm to (191.2, 122.8)
- moved D8 181.0 mm to (175.9, 120.6)
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- renumbered J2 to J3, SW62 to SW25
Connections:
- C1 pad 1: +5V -> GND
- C1 pad 2: GND -> Net-(C2-Pad2)
- C2 pad 1: VBUS -> GND
- C2 pad 2: GND -> Net-(C2-Pad2)
- J1 pad A4: VBUS -> +3.3V
- J1 pad A5: Net-(J1-PadA5) -> unconnected-(J1-PadA5)
- J1 pad A6: D+ -> SPLIT_DATA
- J1 pad A7: D- -> SPLIT_CLOCK
- J1 pad A9: VBUS -> +3.3V
- J1 pad B4: VBUS -> +3.3V
- J1 pad B5: Net-(J1-PadB5) -> unconnected-(J1-PadB5)
- J1 pad B6: D+ -> SPLIT_DATA
- J1 pad B7: D- -> SPLIT_CLOCK
- J1 pad B9: VBUS -> +3.3V
- J1 pad S1: unconnected-(J1-PadS1) -> Net-(C2-Pad2)
- R1 pad 1: Net-(R1-Pad1) -> Net-(C2-Pad2)
- R1 pad 2: Net-(R1-Pad2) -> GND
- R2 pad 1: D+ -> Net-(C2-Pad2)
- R2 pad 2: Net-(R2-Pad2) -> GND
- R3 pad 2: D- -> nRESET
- R4 pad 1: Net-(J1-PadB5) -> Net-(R3-Pad1)
- R4 pad 2: GND -> nRESET
- R5 pad 1: Net-(J1-PadA5) -> SCL
- R5 pad 2: GND -> +3.3V
- R6 pad 1: /QSPI_SS -> SCL
- R7 pad 1: /USBBOOT -> SDA
- R7 pad 2: /QSPI_SS -> +3.3V
- R8 pad 1: GND -> SDA
- R8 pad 2: Net-(D62-Pad1) -> +3.3V
- SW1 pad 2: LED -> ONEWIRE_LED
- SW12 pad 4: Net-(SW18-Pad4) -> Net-(SW12-Pad4)
- SW13 pad 2: Net-(SW25-Pad2) -> Net-(SW12-Pad4)
- SW18 pad 4: Net-(SW30-Pad4) (its old number) -> Net-(SW18-Pad4)
- SW19 pad 2: Net-(SW37-Pad2) -> Net-(SW18-Pad4)
- SW24 pad 4: Net-(SW42-Pad4) -> Net-(SW24-Pad4)
- SW25 pad 2: /nRESET -> Net-(R3-Pad1)
- SW27 pad 2: Net-(SW48-Pad4) -> Net-(SW24-Pad4)
- SW32 pad 4: Net-(SW54-Pad4) -> unconnected-(SW32-Pad4)
- SW7 pad 2: Net-(SW12-Pad4) -> Net-(SW6-Pad4)
- U1 pad 1: +3.3V -> ONEWIRE_LED
- U1 pad 10: +3.3V -> unconnected-(U1-Pad10)
- U1 pad 14: /USBBOOT -> unconnected-(U1-Pad14)
- U1 pad 15: SDA -> unconnected-(U1-Pad15)
- U1 pad 16: SCL -> unconnected-(U1-Pad16)
- U1 pad 19: GND -> unconnected-(U1-Pad19)
- U1 pad 2: unconnected-(U1-Pad2) -> SPLIT_DATA_UART
- U1 pad 20: Net-(U1-Pad20) -> unconnected-(U1-Pad20)
- U1 pad 21: Net-(R1-Pad2) -> +3.3V
- U1 pad 22: +3.3V -> nRESET
- U1 pad 23: +1V1 -> GND
- U1 pad 24: Net-(U1-Pad24) -> unconnected-(U1-Pad24)
- U1 pad 25: Net-(U1-Pad25) -> (no net)
- U1 pad 26: /nRESET -> (no net)
- U1 pad 3: unconnected-(U1-Pad3) -> GND
- U1 pad 4: unconnected-(U1-Pad4) -> GND
- U1 pad 5: unconnected-(U1-Pad5) -> SDA
- U1 pad 6: unconnected-(U1-Pad6) -> SCL

Commit message: mask-2.0.0: first layout prototype
Parts:
- C2, JP2, JP4, R2, R4, R6, R8: moved to B.Cu
- SW32: renamed from SW26; moved to B.Cu
- moved D7 201.7 mm to (39.0, 68.5), turned to 180 degrees
- moved D20 156.7 mm to (56.0, 106.5), turned to 180 degrees
- moved D19 150.0 mm to (40.5, 106.5), turned to 180 degrees
- moved D14 147.3 mm to (57.0, 87.5), turned to 180 degrees
- moved D16 144.1 mm to (96.0, 72.0), turned to 180 degrees
- moved D13 139.5 mm to (36.5, 87.5), turned to 180 degrees
- moved D10 137.0 mm to (94.5, 53.0), turned to 180 degrees
- moved D9 134.9 mm to (76.0, 56.0), turned to 180 degrees
- moved D15 130.4 mm to (76.0, 75.0), turned to 180 degrees
- moved D8 129.9 mm to (57.0, 68.5), turned to 180 degrees
- moved D21 126.5 mm to (83.5, 91.0), turned to 180 degrees
- moved D22 123.8 mm to (93.5, 91.0), turned to 180 degrees
- moved D12 105.7 mm to (133.0, 57.0), turned to 180 degrees
- moved D17 103.8 mm to (115.5, 75.0), turned to 180 degrees
- moved D25 103.4 mm to (87.5, 93.5), turned to 180 degrees
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- renumbered SW27 to SW25, SW28 to SW26, SW29 to SW27, SW30 to SW28, SW31 to SW29, SW32 to SW30, SW25 to SW31
Other:
- board size 307.3 x 148.3 mm -> 143 x 105 mm

Commit message: mask-2.0.0: routing halfway done, 3.3v for led's next
Parts:
- D1, D10, D11, D12, D13, D14, D15, D16, D17, D18, D19, D2, D20, D21, D22, D23, D24, D25, D26, D27, D28, D29, D3, D30, D4, D5, D6, D7, D8, D9: footprint mask:D_SOD-123_TopBottom -> mask:D_0603_1608Metric_TopBottom
- moved JP3 130.7 mm to (153.2, 61.9), turned to 90 degrees
- moved JP4 130.7 mm to (153.2, 61.9), turned to 90 degrees
- moved JP1 116.8 mm to (150.6, 62.5), turned to 90 degrees
- moved JP2 116.8 mm to (150.6, 62.5), turned to 90 degrees
- moved R2 93.1 mm to (158.8, 70.3), turned to -90 degrees
- moved R1 93.1 mm to (158.8, 70.3), turned to -90 degrees
- moved C1 89.1 mm to (160.4, 70.3), turned to 90 degrees
- moved C2 89.1 mm to (160.4, 70.3), turned to 90 degrees
- moved R5 77.6 mm to (151.5, 57.9)
- moved R6 77.6 mm to (151.5, 57.9)
- moved R7 77.0 mm to (151.5, 59.4)
- moved R8 77.0 mm to (151.5, 59.4)
- moved R3 64.6 mm to (208.3, 67.7)
- moved R4 64.6 mm to (208.3, 67.7)
- moved SW31 64.6 mm to (208.3, 72.2)
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Connections:
- D29 pad 1: ROW4 -> ROW3
- D30 pad 1: ROW4 -> ROW3
- SW1 pad 2: ONEWIRE_LED -> Net-(SW2-Pad4)
- SW1 pad 4: Net-(SW1-Pad4) -> Net-(SW7-Pad2)
- SW13 pad 2: Net-(SW12-Pad4) -> Net-(SW14-Pad4)
- SW13 pad 4: Net-(SW13-Pad4) -> Net-(SW19-Pad2)
- SW14 pad 2: Net-(SW13-Pad4) -> Net-(SW15-Pad4)
- SW15 pad 2: Net-(SW14-Pad4) -> Net-(SW15-Pad2)
- SW16 pad 2: Net-(SW15-Pad4) -> Net-(SW17-Pad4)
- SW16 pad 4: Net-(SW16-Pad4) -> Net-(SW15-Pad2)
- SW17 pad 2: Net-(SW16-Pad4) -> Net-(SW18-Pad4)
- SW18 pad 2: Net-(SW17-Pad4) -> Net-(SW12-Pad4)
- SW19 pad 2: Net-(SW18-Pad4) -> Net-(SW19-Pad2)
- SW2 pad 2: Net-(SW1-Pad4) -> Net-(SW2-Pad2)
- SW25 pad 2: Net-(SW24-Pad4) -> Net-(SW26-Pad4)
- SW25 pad 4: Net-(SW25-Pad4) -> unconnected-(SW25-Pad4)
- SW25 pad 5: COL0 -> COL4
- SW26 pad 2: Net-(SW25-Pad4) -> Net-(SW27-Pad4)
- SW26 pad 5: COL1 -> COL5
- SW27 pad 2: Net-(SW26-Pad4) -> Net-(SW28-Pad4)
- SW27 pad 5: COL2 -> COL6
- SW28 pad 2: Net-(SW27-Pad4) -> Net-(SW30-Pad4)
- SW28 pad 5: COL3 -> COL7
- SW29 pad 2: Net-(SW28-Pad4) -> Net-(SW24-Pad4)
- SW29 pad 5: COL4 -> COL6
- SW3 pad 2: Net-(SW2-Pad4) -> Net-(SW4-Pad4)
- SW3 pad 4: Net-(SW3-Pad4) -> Net-(SW2-Pad2)
- SW30 pad 4: unconnected-(SW30-Pad4) -> Net-(SW30-Pad4)
- SW30 pad 5: COL5 -> COL7
- SW4 pad 2: Net-(SW3-Pad4) -> Net-(SW5-Pad4)
- SW5 pad 2: Net-(SW4-Pad4) -> Net-(SW6-Pad4)
- SW6 pad 2: Net-(SW5-Pad4) -> ONEWIRE_LED
- SW7 pad 2: Net-(SW6-Pad4) -> Net-(SW7-Pad2)
Routing:
- net +3.3V: track 0.00 -> 269.6 mm, vias 0 -> 2
- net COL0: track 0.00 -> 192.1 mm, vias 0 -> 5
- net COL1: track 0.00 -> 172.0 mm, vias 0 -> 5
- net COL2: track 0.00 -> 144.1 mm, vias 0 -> 5
- net ROW4: track 0.00 -> 139.7 mm
- net COL4: track 0.00 -> 127.3 mm, vias 0 -> 6
- net COL3: track 0.00 -> 122.9 mm, vias 0 -> 5
- net ROW3: track 0.00 -> 122.0 mm
- net ROW2: track 0.00 -> 111.5 mm
- net COL5: track 0.00 -> 108.3 mm, vias 0 -> 6
- net ROW1: track 0.00 -> 107.5 mm
- net ROW0: track 0.00 -> 101.6 mm, vias 0 -> 4
- net COL7: track 0.00 -> 68.2 mm, vias 0 -> 3
- net COL6: track 0.00 -> 52.7 mm, vias 0 -> 3
- net SPLIT_DATA_UART: track 0.00 -> 43.3 mm, vias 0 -> 1
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- added copper zone on B.Cu, net GND
- added copper zone on F.Cu, net GND
- added copper zone on B.Cu, net Net-(C1-Pad2)
- added copper zone on F.Cu, net Net-(C1-Pad2)
Other:
- board size 143 x 105 mm -> 154 x 106.8 mm
