File: mask-module-0.0.0/mask-module-0.0.0.kicad_sch (KiCad schematic)
At the start: 9 parts, among them J1 Conn_01x02, J2 USB_C_Receptacle_USB2.0, J3 Conn_01x13, J4 Conn_01x13, U1 BQ24075RGT, U2 BMD-340, U3 MCP1703Ax-330xxTT

Commit message: mask-module-0.0.0: update schematic
Parts:
- added C1, C7, C8: 1uF, Capacitor_SMD:C_0402_1005Metric, symbol Device:C_Small
- added C2, C3, C4, C5, C6: 4.7uF, Capacitor_SMD:C_0603_1608Metric, symbol Device:C_Small
- added D1: LED_Small, LED_SMD:LED_0402_1005Metric, symbol Device:LED_Small
- added J3: Conn_ARM_JTAG_SWD_10, Connector:Tag-Connect_TC2050-IDC-NL_2x05_P1.27mm_Vertical, symbol Connector:Conn_ARM_JTAG_SWD_10
- added J4: Conn_01x02, Connector_Molex:Molex_PicoBlade_53261-0271_1x02-1MP_P1.25mm_Horizontal, symbol Connector_Generic:Conn_01x02
- added R3, R4: 10k, Resistor_SMD:R_0402_1005Metric, symbol Device:R_Small
- added R5: 10k / 2k, Resistor_SMD:R_0402_1005Metric, symbol Device:R_Small
- J2: footprint Connector_USB:USB_C_Receptacle_JAE_DX07S016JA1R1500 -> mask:USB_C_Receptacle_GCT_USB4520-xx-x-A_16P_Horizontal
- R1, R2: value 5.11k -> 5.1k; footprint Resistor_SMD:R_0603_1608Metric -> Resistor_SMD:R_0402_1005Metric
- renumbered J3 to J5, J4 to J6
Connections:
- net GND: now also J5.1 (Pin_1), J5.4 (Pin_4), J5.5 (Pin_5), J6.3 (Pin_3), U1.15 (SYSOFF), U1.17 (VSS), U1.4 (~{CE}), U1.5 (EN2), U1.8 (VSS), U2.1 (GND), U2.16 (GND), U2.18 (GND), U2.2 (GND), U2.29 (GND), U2.3 (GND), U2.30 (GND), U2.4 (GND), U2.45 (GND), U2.46 (GND), U2.47 (GND), U2.5 (GND), U2.55 (GND), U3.1 (GND), C1.1, C2.2, C3.2, C4.2, C5.2, C6.2, C7.2, C8.2, J4.2 (Pin_2), R3.2, R5.2
- net VBUS: now also U1.13 (IN), U2.66 (VBUS), C1.2, C4.1
- net P1.00: now reaches J5.10 (Pin_10)
- net P0.11: now reaches J5.11 (Pin_11)
- net P1.04: now reaches J5.12 (Pin_12)
- net P1.06: now reaches J5.13 (Pin_13)
- net P0.06_TXD: now reaches J5.2 (Pin_2)
- net P0.08_RXD: now reaches J5.3 (Pin_3)
- net P0.17: now reaches J5.6 (Pin_6)
- net P0.20: now reaches J5.7 (Pin_7)
- net P0.22: now reaches J5.8 (Pin_8)
- net P0.24: now reaches J5.9 (Pin_9)
- net VDD_NRF: now reaches U2.17 (VCC)
- net VDD_NRF: now also C2.1
- net +5V: now reaches U2.65 (VCCH)
- net +5V: now also J6.2 (Pin_2), U1.10 (OUT), U1.11 (OUT), U1.6 (EN1), U3.3 (VI), C3.1, C6.1, C7.1, R4.1
- net +3V3: now reaches U3.2 (VO)
- net +3V3: now also J6.5 (Pin_5), C8.1
- net at U1.1 (TS): now also R3.1
- net at U1.16 (ISET): now also R5.1
- net VBAT: now reaches U1.2 (BAT), U1.3 (BAT)
- net VBAT: now also J6.1 (Pin_1), C5.1, J4.1 (Pin_1)
- net at U1.9 (~{CHG}): now also D1.1 (K)
- net P1.13: now reaches J6.10 (Pin_10)
- net P1.11: now reaches J6.11 (Pin_11)
- net P0.10: now reaches J6.12 (Pin_12)
- net P0.09: now reaches J6.13 (Pin_13)
- net RESET: now reaches J6.4 (Pin_4)
- net P0.31: now reaches J6.6 (Pin_6)
- net P0.29: now reaches J6.7 (Pin_7)
- net P0.02: now reaches J6.8 (Pin_8)
- net P1.15: now reaches J6.9 (Pin_9)
- new net: D1.2 (A), R4.2
- new net: J3.3 (GND), J3.5 (GND)
- no-connect marks 3 -> 6
Other:
- moved on the sheet: J1

Commit message: module-0.0.0: more shematic work
Parts:
- removed U2: BMD-340, ublox:BMD-340, symbol ublox:BMD-340
- added C10, C9: 1uF, Capacitor_SMD:C_0402_1005Metric, symbol Device:C_Small
- added U4: BMD-380, ublox:BMD-380, symbol ublox:BMD-380
- added Y1: FC-135 32.768KA-A5, Crystal:Crystal_SMD_MicroCrystal_CC7V-T1A-2Pin_3.2x1.5mm, symbol Device:Crystal_Small
Connections:
- net +5V: now also U4.22 (VCCH)
- net D+: now also U4.21 (USB-D+)
- net D-: now also U4.19 (USB-D-)
- net GND: now also J3.3 (GND), J3.5 (GND), C10.2, C9.1, U4.1 (GND), U4.2 (GND), U4.23 (GND), U4.3 (GND), U4.35 (GND), U4.5 (GND), U4.54 (GND), U4.55 (GND), U4.56 (GND), U4.57 (GND), U4.58 (GND), U4.63 (GND)
- net P0.02: now also U4.41 (P0.02/AIN0)
- net P0.06_TXD: now also U4.30 (P0.06)
- net P0.08_RXD: now also U4.29 (P0.08)
- net P0.09: now also U4.53 (P0.09/NFC1)
- net P0.10: now also U4.52 (P0.10/NFC2)
- net P0.11: now also U4.18 (P0.11/TRACEDATA[2])
- net P0.17: now also U4.13 (P0.17)
- net P0.20: now also U4.14 (P0.20)
- net P0.22: now also U4.6 (P0.22)
- net P0.24: now also U4.60 (P0.24)
- net P0.29: now also U4.37 (P0.29/AIN5)
- net P0.31: now also U4.39 (P0.31/AIN7)
- net P1.00: now also U4.11 (SWO/TRACEDATA[0]/P1.00)
- net P1.04: now also U4.48 (P1.03)
- net P1.06: now also U4.50 (P1.06)
- net P1.11: now also U4.51 (P1.11)
- net P1.13: now also U4.47 (P1.13)
- net P1.15: now also U4.40 (P1.15)
- net RESET: now also J3.10 (~{RESET}), U4.12 (P0.18/nRESET)
- net VBUS: now also U4.15 (VBUS)
- net VDD_NRF: now also J3.1 (VTref), U4.24 (VCC)
- net SWDIO: now reaches J3.2 (SWDIO/TMS)
- net SWDIO: now also U4.7 (SWDIO)
- net SWCLK: now reaches J3.4 (SWDCLK/TCK)
- net SWCLK: now also U4.4 (SWCLK)
- new net: C10.1, U4.38 (P0.00/XTAL1), Y1.2
- new net: C9.2, U4.36 (P0.01/XTAL2), Y1.1
- no-connect marks 6 -> 9

Commit message: module-0.0.0: finish pcb
Parts:
- removed J1: Conn_01x02, Connector_JST:JST_PH_S2B-PH-SM4-TB_1x02-1MP_P2.00mm_Horizontal, symbol Connector_Generic:Conn_01x02
- removed J4: Conn_01x02, Connector_Molex:Molex_PicoBlade_53261-0271_1x02-1MP_P1.25mm_Horizontal, symbol Connector_Generic:Conn_01x02
- J2: footprint mask:USB_C_Receptacle_GCT_USB4520-xx-x-A_16P_Horizontal -> Connector_USB:USB_C_Receptacle_JAE_DX07S016JA1R1500
Connections:
- net P0.02: no longer J6.8 (Pin_8)
- net P0.09: now also J5.13 (Pin_13); no longer J6.13 (Pin_13)
- net P0.10: now also J5.12 (Pin_12); no longer J6.12 (Pin_12)
- net P0.11: no longer J5.11 (Pin_11)
- net P0.17: now also J6.10 (Pin_10); no longer J5.6 (Pin_6)
- net P0.20: no longer J5.7 (Pin_7)
- net P0.22: now also J6.13 (Pin_13); no longer J5.8 (Pin_8)
- net P0.24: no longer J5.9 (Pin_9)
- net P0.29: no longer J6.7 (Pin_7)
- net P0.31: no longer J6.6 (Pin_6)
- net P1.00: no longer J5.10 (Pin_10)
- net P1.04: no longer J5.12 (Pin_12)
- net P1.06: now also J5.11 (Pin_11); no longer J5.13 (Pin_13)
- net P1.11: no longer J6.11 (Pin_11)
- net P1.13: no longer J6.10 (Pin_10)
- net P1.15: no longer J6.9 (Pin_9)
- net P0.21: now reaches U4.10 (P0.21)
- net P0.21: now also J6.11 (Pin_11)
- net P0.14: now reaches U4.16 (P0.14)
- net P0.14: now also J6.9 (Pin_9)
- net P0.15: now reaches U4.20 (P0.15)
- net P0.15: now also J6.8 (Pin_8)
- net P0.12: now reaches U4.26 (P0.12/TRACEDATA[1])
- net P0.12: now also J6.7 (Pin_7)
- net P0.07: now reaches U4.27 (P0.07/TRACECLK)
- net P0.07: now also J6.6 (Pin_6)
- net P0.05: now reaches U4.31 (P0.05/AIN3)
- net P0.05: now also J5.6 (Pin_6)
- net P0.27: now reaches U4.32 (P0.27)
- net P0.27: now also J5.7 (Pin_7)
- net P0.26: now reaches U4.33 (P0.26)
- net P0.26: now also J5.8 (Pin_8)
- net P0.04: now reaches U4.34 (P0.04/AIN2)
- net P0.04: now also J5.9 (Pin_9)
- net P1.10: now reaches U4.49 (P1.10)
- net P1.10: now also J5.10 (Pin_10)
- net P0.25: now reaches U4.8 (P0.25)
- net P0.19: now reaches U4.9 (P0.19)
- net P0.19: now also J6.12 (Pin_12)
Other:
- moved on the sheet: C1, C10, C2, C3, C4, C5, C6, C9, D1, J2, J3, R1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
