File: mask-1.1.0/mask-1.1.0.kicad_pcb (KiCad board)
At the start: 2 copper layers, 144.2 x 112.6 mm, 103 parts, among them J1 USB_C_Receptacle_USB2.0, J2 Conn_ARM_JTAG_SWD_10, J3 USB_C_Receptacle_USB2.0, J4 USB_C_Receptacle_USB2.0, J5 JST S2B-PH-SM4, J6 USB_C_Receptacle_USB2.0, SW1 SW_PUSH-MX_W_LED, SW10 SW_PUSH-MX_W_LED, SW11 SW_PUSH-MX_W_LED, SW12 SW_PUSH-MX_W_LED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

Commit message: mask-1.1.0: add 3d models of hotswap sockets on both sides
Routing:
- net unconnected-(SW30B-DOUT-Pad1)_1: track 0.00 -> 4.14 mm, vias 0 -> 1
- net (no net): track 4.14 -> 0.00 mm, vias 1 -> 0
